File: l298_dRIVER/l298_dRIVER.kicad_pcb (KiCad board)
At the start: 2 copper layers, 32 parts, among them J1 Screw_Terminal_01x02, J2 Current_Sense, J3 Signal A, J4 Signal B, J5 Screw_Terminal_01x02, J6 Screw_Terminal_01x02, J7 +5V, J8 gnd, U1 L298HN, U2 L7805

Commit message: l298_driver completed
Parts:
- U1: footprint kicad-library:TO-220-15_P2.54x2.54mm_StaggerOdd_Lead4.58mm_Vertical_with_heatsink -> Package_TO_SOT_THT:TO-220-15_P2.54x2.54mm_StaggerOdd_Lead4.58mm_Vertical
- moved U2 126.5 mm to (120.2, 139.9), turned to 270 degrees
- moved C4 126.4 mm to (117.5, 140.8), turned to 270 degrees
- moved J7 111.3 mm to (91.4, 139.2), turned to 270 degrees
- moved C5 105.3 mm to (94.5, 140.9), turned to 270 degrees
- moved R3 100.5 mm to (88.7, 141.7), turned to 180 degrees
- moved J8 98.4 mm to (81.1, 144.1), turned to 90 degrees
- moved D10 89.1 mm to (77.2, 144.3), turned to 90 degrees
- moved J1 70.1 mm to (141.3, 146.4), turned to 90 degrees
- moved D1 53.2 mm to (138.8, 136.0), turned to 0 degrees
- moved C1 46.6 mm to (129.6, 141.9), turned to 270 degrees
- moved J5 45.7 mm to (73.2, 126.1), turned to 270 degrees
- moved J6 39.7 mm to (141.1, 131.4), turned to 90 degrees
- moved C2 38.2 mm to (93.8, 121.8), turned to 270 degrees
- moved C3 37.9 mm to (119.9, 122.0), turned to 270 degrees
- moved D9 34.6 mm to (133.3, 131.9), turned to 90 degrees
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Routing:
- net VCC: track 60.0 -> 293.6 mm
- net GND: track 46.5 -> 102.9 mm, vias 0 -> 2
- net +5V: track 0.00 -> 46.6 mm
- net Net-(D2-Pad2): track 58.4 -> 29.5 mm
- net Net-(D4-Pad2): track 87.2 -> 62.5 mm
- net /S2: track 0.00 -> 23.9 mm, vias 0 -> 2
- net Net-(J4-Pad2): track 0.00 -> 23.4 mm
- net Net-(J4-Pad3): track 0.00 -> 11.8 mm
- net Net-(J4-Pad1): track 0.00 -> 11.2 mm
- net Net-(J3-Pad3): track 0.00 -> 10.7 mm
- net Net-(J3-Pad1): track 0.70 -> 11.2 mm
- net Net-(J3-Pad2): track 0.00 -> 8.61 mm
- net Net-(D8-Pad2): track 49.4 -> 40.8 mm
- net /S1: track 0.00 -> 8.02 mm
- net Net-(D6-Pad2): track 51.9 -> 48.0 mm
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- added copper zone on B.Cu, net GND
Other:
- board outline added: 82 x 34.1 mm
- board text added: "2k19"
- board text added: "SWCPPR"
